File: busboard10/busboard10.kicad_pcb (KiCad board)
At the start: 2 copper layers, 200 x 25 mm, 18 parts, among them J1 Synth_power_2x5_narrow, J10 Synth_power_2x5_narrow, J11 Synth_power_2x5_narrow, J12 Synth_power_2x5_narrow, J13 Conn_01x03, J2 Synth_power_2x5_narrow, J3 Synth_power_2x5_narrow, J4 Synth_power_2x5_narrow, J5 Synth_power_2x5_narrow, J6 Synth_power_2x5_narrow, J7 Synth_power_2x5_narrow, J8 Synth_power_2x5_narrow, J9 Synth_power_2x5_narrow

Commit message: anal centering
Parts:
- moved G*** 0.50 mm to (56.2, 62.5)
- moved J13 0.50 mm to (47.5, 62.5)
Changed lines of the file:
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@@
   )
   (module busboard10:analogoutput_8mm locked (layer F.Cu)
-    (at 56.25 62)
+    (at 56.25 62.5)
     (fp_text reference G*** (at 0 0) (layer F.SilkS) hide
       (effects (font (size 1.524 1.524) (thickness 0.3)))
@@
   )
   (module ao_tht:TerminalBlock_Degson_DG301_1x03_P5.00mm_Vertical (layer F.Cu)
-    (at 47.5 62 270)
+    (at 47.5 62.5 270)
     (descr "terminal block RND 205-00079, vertical (cable from top), 3 pins, pitch 5mm, size 15x10mm^2, drill diamater 1.3mm, pad diameter 2.5mm, see http://cdn-reichelt.de/documents/datenblatt/C151/RND_205-00276_DB_EN.pdf, script-generated with , script-generated using https://github.com/pointhi/kicad-footprint-generator/scripts/TerminalBlock_RND")
     (tags "THT terminal block RND 205-00079 vertical pitch 5mm size 15x10mm^2 drill 1.3mm pad 2.5mm")
@@
   )
   (gr_line (start 242 75) (end 42 75) (layer Edge.Cuts) (width 0.15))
-  (gr_text GND (at 51.5 60.5 90) (layer F.SilkS)
+  (gr_text GND (at 51.5 61 90) (layer F.SilkS)
     (effects (font (size 1 1) (thickness 0.2)) (justify right))
   )
-  (gr_text +12V (at 51.5 65 90) (layer F.SilkS)
+  (gr_text +12V (at 51.5 65.5 90) (layer F.SilkS)
     (effects (font (size 1 1) (thickness 0.2)) (justify right))
   )
-  (gr_text -12V (at 51.5 55 90) (layer F.SilkS)
+  (gr_text -12V (at 51.5 55.5 90) (layer F.SilkS)
     (effects (font (size 1 1) (thickness 0.2)) (justify right))
   )
@@
     (polygon
       (pts
-        (xy 41.5 48.5) (xy 41.5 61.5) (xy 242.5 61.5) (xy 242.5 48.5)
+        (xy 41.5 48.5) (xy 41.5 62) (xy 242.5 62) (xy 242.5 48.5)
       )
     )
@@
     (polygon
       (pts
-        (xy 41.5 62.5) (xy 41.5 82.5) (xy 242.5 82.5) (xy 242.5 62.5)
+        (xy 41.5 63) (xy 41.5 82.5) (xy 242.5 82.5) (xy 242.5 63)
       )
     )
